Commit message: Add files via upload

File: manipulator/urdf/models.urdf (robot description, URDF)
Before this commit: robot robot_manipulator, 7 links, 6 joints
Joints:
- joint joint_1: limit lower=-2.967 upper=2.967 effort=0 velocity=1.7453 -> lower=-2.967 upper=2.967 effort=10.0 velocity=1.7453; origin xyz=0 0 0 rpy=0 0 0 -> xyz=0 0 0.1255 rpy=0 0 0
- joint joint_2: limit lower=-1.134 upper=1.4855 effort=0 velocity=1.5707 -> lower=-1.134 upper=1.4855 effort=10.0 velocity=1.5707; origin xyz=0 0 0 rpy=0 0 0 -> xyz=0.15 -0.137 0.361 rpy=0 0 0
- joint joint_3: limit lower=-3.142 upper=1.222 effort=0 velocity=1.5707 -> lower=-3.142 upper=1.222 effort=10.0 velocity=1.5707; origin xyz=0 0 0 rpy=0 0 0 -> xyz=0 0.03 0.7 rpy=0 0 0
- joint joint_4: limit lower=-5.236 upper=5.236 effort=0 velocity=2.9671 -> lower=-5.236 upper=5.236 effort=10.0 velocity=2.9671; origin xyz=0 0 0 rpy=0 0 0 -> xyz=0.314 0.107 0 rpy=0 0 0
- joint joint_5: limit lower=-2.094 upper=2.094 effort=0 velocity=2.4435 -> lower=-2.094 upper=2.094 effort=10.0 velocity=2.4435; origin xyz=0 0 0 rpy=0 0 0 -> xyz=0.286 0 0 rpy=0 0 0
- joint joint_6: limit lower=-6.283 upper=6.283 effort=0 velocity=3.3161 -> lower=-6.283 upper=6.283 effort=10.0 velocity=3.3161; origin xyz=0 0 0 rpy=0 0 0 -> xyz=0.033 0 0 rpy=0 0 0
